File: levelshuifter.sch (KiCad schematic (older format))
At the start: 31 parts, among them J1 Screw_Terminal_01x02, J2 Conn_02x20_Odd_Even, J3 Conn_02x08_Odd_Even, J4 Conn_02x08_Odd_Even, J5 Conn_02x08_Odd_Even, U1 LM1117-3.3, U2 74LVC8T245PW, U3 74LVC8T245PW, U4 74LVC8T245PW, U5 L7805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

Commit message: anotaciones solucionadas
Other:
- note added: "ENTRADA DE1SoC\n"
- note added: "SALIDA MATRICES LED\n"
Changed lines of the file:
@@
 	1    0    0    -1
 $EndComp
+Text Notes 1000 3650 0    79   ~ 0
+ENTRADA DE1SoC\n
+Text Notes 6250 850  0    79   ~ 0
+SALIDA MATRICES LED\n
+Text Notes 6200 3350 0    79   ~ 0
+SALIDA MATRICES LED\n
+Text Notes 9550 700  0    79   ~ 0
+SALIDA MATRICES LED\n
 $EndSCHEMATC

Commit message: cambios 2
Parts:
- C1, C11, C7, C8: symbol Device:CP -> levelshuifter-rescue:CP-Device
- C10, C12, C13, C2, C3, C4, C5, C6, C9: symbol Device:C -> levelshuifter-rescue:C-Device
- FID1, FID2: symbol Mechanical:Fiducial -> levelshuifter-rescue:Fiducial-Mechanical
- H1, H2, H3, H4: symbol Mechanical:MountingHole -> levelshuifter-rescue:MountingHole-Mechanical
- J1: symbol Connector:Screw_Terminal_01x02 -> levelshuifter-rescue:Screw_Terminal_01x02-Connector
- J2: symbol Connector_Generic:Conn_02x20_Odd_Even -> levelshuifter-rescue:Conn_02x20_Odd_Even-Connector_Generic
- J3, J4, J5: symbol Connector_Generic:Conn_02x08_Odd_Even -> levelshuifter-rescue:Conn_02x08_Odd_Even-Connector_Generic
- U1: symbol Regulator_Linear:LM1117-3.3 -> levelshuifter-rescue:LM1117-3.3-Regulator_Linear
- U2, U3, U4, U6, U7: symbol levelshuifter-rescue:74LVC8T245PW-74LVC8T245PW -> levelshuifter-rescue:74LVC8T245PW-74LVC8T245PW-levelshuifter-rescue
- U5: symbol Regulator_Linear:L7805 -> levelshuifter-rescue:L7805-Regulator_Linear
