File: levelshuifter.kicad_pcb (KiCad board)
At the start: 2 copper layers, 55 x 153 mm, 30 parts, among them J1 Screw_Terminal_01x02, J2 Conn_02x20_Odd_Even, J3 Conn_02x08_Odd_Even, J4 Conn_02x08_Odd_Even, J5 Conn_02x08_Odd_Even, U1 LM1117-3.3, U2 74LVC8T245PW, U3 74LVC8T245PW, U4 74LVC8T245PW, U5 L7805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

Commit message: anotaciones solucionadas
Parts:
- moved C11 32.3 mm to (45.7, 163.2), turned to 270 degrees
- moved C12 31.1 mm to (61.8, 150.3)
- moved C3 31.1 mm to (61.8, 107.2)
- moved C4 31.1 mm to (61.8, 73.7)
- moved C5 31.1 mm to (61.8, 47.2)
- moved C6 31.1 mm to (61.8, 125.5)
- moved U1 31.1 mm to (50.7, 47.1)
- moved U2 31.1 mm to (61.8, 113.8)
- moved U3 31.1 mm to (61.8, 53.9)
- moved U4 31.1 mm to (61.8, 79.8)
- moved U5 31.1 mm to (36.9, 47.5)
- moved U6 31.1 mm to (61.8, 131.6)
- moved C1 31.1 mm to (62.5, 41.9)
- moved C10 31.1 mm to (30.6, 139.3)
- moved C13 31.1 mm to (50.5, 33.1)
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Other:
- board text added: "2020"
- board text added: "Fabricante seleccionado: Microcircuitos (Colombia) Limitaciones: https://pcbmicrocircuitos.com/wp-content/uploads/2016/12/medidas-minimas-microcircuitos-1.jpg Distancias: cobre-cobre: 0.203mm agujero-agujero:0.5mm pads-serigraf:0.23mm Ancho: Pista:0.203mm Via:0.25mm Serigrafía:0.23mm"
- board text added: "HE-2903-01-08 SERIE:"
